File: PCB/PCB_ESP32/PCH_ESP32.kicad_pcb (KiCad board)
At the start: 2 copper layers, 72 x 46.5 mm, 10 parts, among them J1 Conn_01x16_Pin, J2 Conn_01x16_Pin

Commit message: new pcb model
Parts:
- added REF**: MountingHole_3.2mm_M3, MountingHole:MountingHole_3.2mm_M3, F.Cu at (125.5, 52.5)
- added REF**: MountingHole_3.2mm_M3, MountingHole:MountingHole_3.2mm_M3, F.Cu at (125.5, 101.0)
- added REF**: MountingHole_3.2mm_M3, MountingHole:MountingHole_3.2mm_M3, F.Cu at (199.5, 101.0)
- added REF**: MountingHole_3.2mm_M3, MountingHole:MountingHole_3.2mm_M3, F.Cu at (199.5, 52.5)
Other:
- board size 72 x 46.5 mm -> 85 x 59.5 mm
- board text added: "ELIADE ELI-NP HeatMap"
- board text added: "GND"
- board text added: "SCL"
- board text added: "SDA"
- board text added: "VCC"
- board text removed: "Eliade"
