File: PCB/PCB/PCH_ESP32.kicad_sch (KiCad schematic)
At the start: 18 parts, among them J1 Conn_01x16_Pin, J2 Conn_01x16_Pin

Commit message: added the new pcb design, and fixel the code to write real values
Parts:
- J1, J2: symbol Connector:Conn_01x16_Pin -> Connector:Conn_01x15_Pin
- renumbered S5 to S1, S6 to S2, S7 to S3, S8 to S4, S1 to S5, S2 to S6, S3 to S7, S4 to S8
Connections:
- net at J1.15 (Pin_15): now also S8.4 (Pin_4)
- net at J2.11 (Pin_11): no longer S8.4 (Pin_4)
Changed lines of the file:
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@@
+	(wire
+		(pts
+			(xy 76.2 119.38) (xy 129.54 119.38)
+		)
+		(stroke
+			(width 0)
+			(type default)
+		)
+	)
 	(wire
 		(pts
@@
 	(wire
 		(pts
-			(xy 111.76 119.38) (xy 129.54 119.38)
-		)
-		(stroke
-			(width 0)
-			(type default)
-		)
-	)
-	(wire
-		(pts
 			(xy 133.35 115.57) (xy 133.35 123.19)
 		)
@@
 	(wire
 		(pts
+			(xy 76.2 119.38) (xy 76.2 107.95)
+		)
+		(stroke
+			(width 0)
+			(type default)
+		)
+	)
+	(wire
+		(pts
 			(xy 44.45 91.44) (xy 44.45 92.71)
 		)
@@
 	(wire
 		(pts
-			(xy 111.76 99.06) (xy 111.76 119.38)
-		)
-		(stroke
-			(width 0)
-			(type default)
-		)
-	)
-	(wire
-		(pts
 			(xy 111.76 147.32) (xy 111.76 143.51)
 		)
@@
 	(wire
 		(pts
-			(xy 100.33 99.06) (xy 111.76 99.06)
-		)
-		(stroke
-			(width 0)
-			(type default)
-		)
-	)
-	(wire
-		(pts
 			(xy 52.07 93.98) (xy 76.2 93.98)
 		)
@@
 		(pts
 			(xy 99.06 82.55) (xy 99.06 81.28)
-		)
-		(stroke
-			(width 0)
-			(type default)
-		)
-	)
-	(wire
-		(pts
-			(xy 100.33 99.06) (xy 100.33 97.79)
 		)
 		(stroke
@@
 		(on_board yes)
 		(dnp no)
-		(property "Reference" "S8"
+		(property "Reference" "S4"
 			(at 44.958 119.888 0)
 			(effects
@@
 			(project ""
 				(path "/f0f054d5-4ad3-45c7-9534-a66f7d04443f"
-					(reference "S8")
+					(reference "S4")
 					(unit 1)
 				)
@@
 	)
 	(symbol
-		(lib_name "Conn_01x04_Pin_1")
 		(lib_id "Connector:Conn_01x04_Pin")
 		(at 49.53 74.93 0)
@@
 		(on_board yes)
 		(dnp no)
-		(property "Reference" "S5"
+		(property "Reference" "S1"
 			(at 45.466 82.55 0)
 			(effects
@@
 			(project ""
 				(path "/f0f054d5-4ad3-45c7-9534-a66f7d04443f"
-					(reference "S5")
+					(reference "S1")
 					(unit 1)
 				)
@@
 	)
 	(symbol
-		(lib_name "Conn_01x16_Pin_1")
-		(lib_id "Connector:Conn_01x16_Pin")
+		(lib_id "Connector:Conn_01x15_Pin")
 		(at 71.12 90.17 0)
 		(unit 1)
@@
 			)
 		)
-		(property "Description" "Generic connector, single row, 01x16, script generated"
+		(property "Description" "Generic connector, single row, 01x15, script generated"
 			(at 71.12 90.17 0)
 			(effects
@@
 		(pin "1"
 		)
+		(pin "2"
+		)
+		(pin "3"
+		)
+		(pin "4"
+		)
+		(pin "5"
+		)
+		(pin "6"
+		)
+		(pin "7"
+		)
+		(pin "15"
+		)
+		(pin "8"
+		)
+		(pin "9"
+		)
 		(pin "10"
 		)
-		(pin "9"
-		)
-		(pin "4"
+		(pin "11"
+		)
+		(pin "12"
 		)
 		(pin "13"
 		)
-		(pin "16"
-		)
-		(pin "12"
-		)
-		(pin "11"
-		)
-		(pin "15"
-		)
 		(pin "14"
-		)
-		(pin "2"
-		)
-		(pin "3"
-		)
-		(pin "5"
-		)
-		(pin "7"
-		)
-		(pin "6"
-		)
-		(pin "8"
 		)
 		(instances
@@
 		(on_board yes)
 		(dnp no)
-		(property "Reference" "S7"
+		(property "Reference" "S3"
 			(at 45.466 106.934 0)
 			(effects
@@
 			(project ""
 				(path "/f0f054d5-4ad3-45c7-9534-a66f7d04443f"
-					(reference "S7")
+					(reference "S3")
 					(unit 1)
 				)
@@
 		(on_board yes)
 		(dnp no)
-		(property "Reference" "S2"
+		(property "Reference" "S6"
 			(at 127.762 95.504 0)
 			(effects
@@
 			(project ""
 				(path "/f0f054d5-4ad3-45c7-9534-a66f7d04443f"
-					(reference "S2")
+					(reference "S6")
 					(unit 1)
 				)
@@
 		(on_board yes)
 		(dnp no)
-		(property "Reference" "S1"
+		(property "Reference" "S5"
 			(at 127.508 82.55 0)
 			(effects
@@
 			(project ""
 				(path "/f0f054d5-4ad3-45c7-9534-a66f7d04443f"
-					(reference "S1")
+					(reference "S5")
 					(unit 1)
 				)
@@
 		(on_board yes)
 		(dnp no)
-		(property "Reference" "S4"
+		(property "Reference" "S8"
 			(at 128.016 122.428 0)
 			(effects
@@
 			(project ""
 				(path "/f0f054d5-4ad3-45c7-9534-a66f7d04443f"
-					(reference "S4")
+					(reference "S8")
 					(unit 1)
 				)
@@
 		(on_board yes)
 		(dnp no)
-		(property "Reference" "S3"
+		(property "Reference" "S7"
 			(at 127.762 108.204 0)
 			(effects
@@
 			(project ""
 				(path "/f0f054d5-4ad3-45c7-9534-a66f7d04443f"
-					(reference "S3")
+					(reference "S7")
 					(unit 1)
 				)
@@
 	)
 	(symbol
-		(lib_name "Conn_01x04_Pin_2")
 		(lib_id "Connector:Conn_01x04_Pin")
 		(at 49.53 87.63 0)
@@
 		(on_board yes)
 		(dnp no)
-		(property "Reference" "S6"
+		(property "Reference" "S2"
 			(at 45.212 94.488 0)
 			(effects
@@
 			(project ""
 				(path "/f0f054d5-4ad3-45c7-9534-a66f7d04443f"
-					(reference "S6")
+					(reference "S2")
 					(unit 1)
 				)
@@
 	)
 	(symbol
-		(lib_id "Connector:Conn_01x16_Pin")
+		(lib_id "Connector:Conn_01x15_Pin")
 		(at 105.41 90.17 0)
 		(mirror y)
@@
 			)
 		)
-		(property "Description" "Generic connector, single row, 01x16, script generated"
+		(property "Description" "Generic connector, single row, 01x15, script generated"
 			(at 105.41 90.17 0)
 			(effects
@@
 		(pin "1"
 		)
+		(pin "2"
+		)
+		(pin "3"
+		)
+		(pin "4"
+		)
+		(pin "13"
+		)
+		(pin "12"
+		)
+		(pin "5"
+		)
+		(pin "6"
+		)
+		(pin "14"
+		)
+		(pin "7"
+		)
+		(pin "8"
+		)
+		(pin "9"
+		)
 		(pin "10"
 		)
-		(pin "9"
-		)
-		(pin "4"
-		)
-		(pin "13"
-		)
-		(pin "16"
-		)
-		(pin "12"
-		)
 		(pin "11"
 		)
 		(pin "15"
 		)
-		(pin "14"
-		)
-		(pin "2"
-		)
-		(pin "3"
-		)
-		(pin "5"
-		)
-		(pin "7"
-		)
-		(pin "6"
-		)
-		(pin "8"
-		)
 		(instances
